Commit message: IK code with PWM modifications for pi

File: arm_code_logitech/src/description/urdf/four_dof_arm.urdf.xacro (robot description, xacro)
@@ -1,14 +1,11 @@
 <?xml version="1.0"?>
 <robot xmlns:xacro="http://www.ros.org/wiki/xacro" name="four_dof_arm">
-  <!-- Shared 4-DOF model. Keep the original visual layout and the original
-       joint-axis convention: each joint rotates about the axis of the link
-       that proceeds from it. -->
+  <!-- Robot geometry placeholders.
+       Swap mesh filenames to your exported SLDPRT->(dae/stl) paths. -->
   <xacro:include filename="$(find arm_description)/urdf/ros2_control.xacro"/>
   <xacro:arg name="controllers_file" default="$(find arm_config)/config/ros2_controllers.yaml"/>
-  <xacro:arg name="initial_positions_file" default="$(find arm_config)/config/initial_positions.yaml"/>
-  <xacro:property name="mesh_dir" value="$(find arm_description)/meshes"/>
+  <xacro:property name="mesh_dir" value="package://arm_description/meshes"/>
   <xacro:property name="controllers_file_path" value="$(arg controllers_file)"/>
-  <xacro:property name="initial_positions_file_path" value="$(arg initial_positions_file)"/>
-  <!-- Basic link dimensions -->
+  <!-- Basic link dimensions (scaled 10x) -->
   <xacro:property name="link1_length" value="1.27"/>
   <xacro:property name="link2_length" value="1.27"/>
@@ -16,4 +13,6 @@
   <!-- Convert millimeter-based meshes to meters and scale 10x -->
   <xacro:property name="mesh_scale" value="0.01 0.01 0.01"/>
+  <!-- Placeholder meshes are already in metric scale -->
+  <xacro:property name="placeholder_scale" value="1.0 1.0 1.0"/>
   <xacro:macro name="default_inertial" params="mass">
     <inertial>
@@ -44,6 +43,6 @@
   </link>
   <joint name="joint1" type="revolute">
-    <origin xyz="0 0 0.10" rpy="0 0 0"/>
-    <axis xyz="0 0 -1"/>
+    <origin xyz="0 0 0.10" rpy="0 0 0"/> <!-- Place joint1 above base top; links hang below -->
+    <axis xyz="0 0 -1"/> <!-- roll link1 about its long axis -->
     <parent link="base_link"/>
     <child link="link1"/>
@@ -55,5 +54,5 @@
       <origin xyz="0 0 -0.635" rpy="0 0 0"/>
       <geometry>
-        <box size="0.14 0.14 ${link1_length}"/>
+        <box size="0.10 0.10 1.27"/>
       </geometry>
       <material name="blue">
@@ -62,7 +61,7 @@
     </visual>
     <collision>
-      <origin xyz="0 0 -0.635" rpy="0 0 0"/>
+      <origin xyz="0 0 0" rpy="0 0 0"/>
       <geometry>
-        <box size="0.14 0.14 ${link1_length}"/>
+        <sphere radius="0.01"/>
       </geometry>
     </collision>
@@ -70,6 +69,6 @@
   </link>
   <joint name="joint2" type="revolute">
-    <origin xyz="0 0 -${link1_length}" rpy="0 0 0"/>
-    <axis xyz="1 0 0"/>
+    <origin xyz="0 0 -${link1_length}" rpy="0 0 0"/> <!-- end of link1 -->
+    <axis xyz="1 0 0"/> <!-- roll link2 about its long axis (+X) -->
     <parent link="link1"/>
     <child link="link2"/>
@@ -79,7 +78,7 @@
   <link name="link2">
     <visual>
-      <origin xyz="${link2_length / 2.0} 0 0" rpy="0 0 0"/>
+      <origin xyz="0.635 0 0" rpy="0 0 0"/>
       <geometry>
-        <box size="${link2_length} 0.14 0.14"/>
+        <box size="1.27 0.10 0.10"/>
       </geometry>
       <material name="light_grey">
@@ -88,7 +87,7 @@
     </visual>
     <collision>
-      <origin xyz="${link2_length / 2.0} 0 0" rpy="0 0 0"/>
+      <origin xyz="0 0 0" rpy="0 0 0"/>
       <geometry>
-        <box size="${link2_length} 0.14 0.14"/>
+        <sphere radius="0.01"/>
       </geometry>
     </collision>
@@ -96,6 +95,6 @@
   </link>
   <joint name="joint3" type="revolute">
-    <origin xyz="${link2_length} 0 0" rpy="0 0 0"/>
-    <axis xyz="0 0 -1"/>
+    <origin xyz="${link2_length} 0 0" rpy="0 0 0"/> <!-- end of link2 -->
+    <axis xyz="0 0 -1"/> <!-- roll link3 about its long axis (-Z) -->
     <parent link="link2"/>
     <child link="link3"/>
@@ -107,5 +106,5 @@
       <origin xyz="0 0 -0.635" rpy="0 0 0"/>
       <geometry>
-        <box size="0.12 0.12 ${link3_length}"/>
+        <box size="0.10 0.10 1.27"/>
       </geometry>
       <material name="blue">
@@ -114,7 +113,7 @@
     </visual>
     <collision>
-      <origin xyz="0 0 -0.635" rpy="0 0 0"/>
+      <origin xyz="0 0 0" rpy="0 0 0"/>
       <geometry>
-        <box size="0.12 0.12 ${link3_length}"/>
+        <sphere radius="0.01"/>
       </geometry>
     </collision>
@@ -157,27 +156,6 @@
       </material>
     </visual>
-    <collision>
-      <origin xyz="0.8 0 0" rpy="0 0 0"/>
-      <geometry>
-        <box size="1.2 0.8 0.4"/>
-      </geometry>
-    </collision>
-    <collision>
-      <origin xyz="1.4 0.4 0" rpy="0 0 0"/>
-      <geometry>
-        <box size="1.4 0.2 0.4"/>
-      </geometry>
-    </collision>
-    <collision>
-      <origin xyz="1.4 -0.4 0" rpy="0 0 0"/>
-      <geometry>
-        <box size="1.4 0.2 0.4"/>
-      </geometry>
-    </collision>
     <xacro:default_inertial mass="0.5"/>
   </link>
-  <xacro:ros2_control_block
-    controllers_file="${controllers_file_path}"
-    initial_positions_file="${initial_positions_file_path}"
-  />
+  <xacro:ros2_control_block controllers_file="${controllers_file_path}"/>
 </robot>

File: arm_code_logitech/src/description/urdf/ros2_control.xacro (robot description, xacro)
@@ -1,6 +1,5 @@
 <?xml version="1.0"?>
 <robot xmlns:xacro="http://www.ros.org/wiki/xacro">
-  <xacro:macro name="ros2_control_block" params="controllers_file initial_positions_file">
-    <xacro:property name="initial_positions" value="${xacro.load_yaml(initial_positions_file)['arm']}"/>
+  <xacro:macro name="ros2_control_block" params="controllers_file">
     <ros2_control name="four_dof_arm_system" type="system">
       <hardware>
@@ -10,28 +9,20 @@
       <joint name="joint1">
         <command_interface name="position"/>
-        <state_interface name="position">
-          <param name="initial_value">${initial_positions['joint1']}</param>
-        </state_interface>
+        <state_interface name="position"/>
         <state_interface name="velocity"/>
       </joint>
       <joint name="joint2">
         <command_interface name="position"/>
-        <state_interface name="position">
-          <param name="initial_value">${initial_positions['joint2']}</param>
-        </state_interface>
+        <state_interface name="position"/>
         <state_interface name="velocity"/>
       </joint>
       <joint name="joint3">
         <command_interface name="position"/>
-        <state_interface name="position">
-          <param name="initial_value">${initial_positions['joint3']}</param>
-        </state_interface>
+        <state_interface name="position"/>
         <state_interface name="velocity"/>
       </joint>
       <joint name="joint4">
         <command_interface name="position"/>
-        <state_interface name="position">
-          <param name="initial_value">${initial_positions['joint4']}</param>
-        </state_interface>
+        <state_interface name="position"/>
         <state_interface name="velocity"/>
       </joint>
